Commit message: working simulation of the robot (torso only)

File: data/talos.urdf (robot description, URDF)
Before this commit: robot talos, 82 links, 81 joints
Links:
- removed link gripper_left_base_link
- removed link gripper_left_fingertip_1_dummy_mimic_link
- removed link gripper_left_fingertip_1_link
- removed link gripper_left_fingertip_2_dummy_mimic_link
- removed link gripper_left_fingertip_2_link
- removed link gripper_left_fingertip_3_dummy_mimic_link
- removed link gripper_left_fingertip_3_link
- removed link gripper_left_inner_double_dummy_mimic_link
- removed link gripper_left_inner_double_link
- removed link gripper_left_inner_single_dummy_mimic_link
- removed link gripper_left_inner_single_link
- removed link gripper_left_link_dummy_mimic_link
- removed link gripper_left_motor_double_link
- removed link gripper_left_motor_single_dummy_mimic_link
- removed link gripper_left_motor_single_link
- removed link gripper_right_base_link
- removed link gripper_right_fingertip_1_dummy_mimic_link
- removed link gripper_right_fingertip_1_link
- removed link gripper_right_fingertip_2_dummy_mimic_link
- removed link gripper_right_fingertip_2_link
- removed link gripper_right_fingertip_3_dummy_mimic_link
- removed link gripper_right_fingertip_3_link
- removed link gripper_right_inner_double_dummy_mimic_link
- removed link gripper_right_inner_double_link
- removed link gripper_right_inner_single_dummy_mimic_link
- removed link gripper_right_inner_single_link
- removed link gripper_right_link_dummy_mimic_link
- removed link gripper_right_motor_double_link
- removed link gripper_right_motor_single_dummy_mimic_link
- removed link gripper_right_motor_single_link
- removed link left_foot_lower_left
- removed link left_foot_lower_right
- removed link left_foot_upper_left
- removed link left_foot_upper_right
- removed link left_sole_link
- removed link leg_left_1_link
- removed link leg_left_2_link
- removed link leg_left_3_link
- removed link leg_left_4_link
- removed link leg_left_5_link
- removed link leg_left_6_link
- removed link leg_right_1_link
- removed link leg_right_2_link
- removed link leg_right_3_link
- removed link leg_right_4_link
- removed link leg_right_5_link
- removed link leg_right_6_link
- removed link right_foot_lower_left
- removed link right_foot_lower_right
- removed link right_foot_upper_left
- removed link right_foot_upper_right
- removed link right_sole_link
- removed link wrist_left_ft_tool_link
Joints:
- removed joint gripper_left_base_link_joint
- removed joint gripper_left_fingertip_1_joint
- removed joint gripper_left_fingertip_1_joint_mimic
- removed joint gripper_left_fingertip_2_joint
- removed joint gripper_left_fingertip_2_joint_mimic
- removed joint gripper_left_fingertip_3_joint
- removed joint gripper_left_fingertip_3_joint_mimic
- removed joint gripper_left_inner_double_joint
- removed joint gripper_left_inner_double_joint_mimic
- removed joint gripper_left_inner_single_joint
- removed joint gripper_left_inner_single_joint_mimic
- removed joint gripper_left_joint
- removed joint gripper_left_link_joint_mimic
- removed joint gripper_left_motor_single_joint
- removed joint gripper_left_motor_single_joint_mimic
- removed joint gripper_right_base_link_joint
- removed joint gripper_right_fingertip_1_joint
- removed joint gripper_right_fingertip_1_joint_mimic
- removed joint gripper_right_fingertip_2_joint
- removed joint gripper_right_fingertip_2_joint_mimic
- removed joint gripper_right_fingertip_3_joint
- removed joint gripper_right_fingertip_3_joint_mimic
- removed joint gripper_right_inner_double_joint
- removed joint gripper_right_inner_double_joint_mimic
- removed joint gripper_right_inner_single_joint
- removed joint gripper_right_inner_single_joint_mimic
- removed joint gripper_right_joint
- removed joint gripper_right_link_joint_mimic
- removed joint gripper_right_motor_single_joint
- removed joint gripper_right_motor_single_joint_mimic
- removed joint left_foot_lower_left_fix_joint
- removed joint left_foot_lower_right_fix_joint
- removed joint left_foot_upper_left_fix_joint
- removed joint left_foot_upper_right_fix_joint
- removed joint leg_left_1_joint
- removed joint leg_left_2_joint
- removed joint leg_left_3_joint
- removed joint leg_left_4_joint
- removed joint leg_left_5_joint
- removed joint leg_left_6_joint
- removed joint leg_left_sole_fix_joint
- removed joint leg_right_1_joint
- removed joint leg_right_2_joint
- removed joint leg_right_3_joint
- removed joint leg_right_4_joint
- removed joint leg_right_5_joint
- removed joint leg_right_6_joint
- removed joint leg_right_sole_fix_joint
- removed joint right_foot_lower_left_fix_joint
- removed joint right_foot_lower_right_fix_joint
- removed joint right_foot_upper_left_fix_joint
- removed joint right_foot_upper_right_fix_joint
- removed joint wrist_left_tool_joint

Commit message: full robot (without fingertip, not working with pinocchio)

File: data/talos.urdf (robot description, URDF)
Before this commit: robot talos, 29 links, 28 joints
Links:
- added link gripper_left_base_link, mass 0.637534; collision cylinder length=0.026984385527609595 radius=0.060646620008233225; collision sphere radius=0.060646620008233225
- added link gripper_left_fingertip_1_dummy_mimic_link
- added link gripper_left_fingertip_2_dummy_mimic_link
- added link gripper_left_fingertip_3_dummy_mimic_link
- added link gripper_left_inner_double_dummy_mimic_link
- added link gripper_left_inner_double_link, mass 0.087986; collision cylinder length=0.03702274994466908 radius=0.04877941290859063; collision sphere radius=0.04877941290859063
- added link gripper_left_inner_single_dummy_mimic_link
- added link gripper_left_inner_single_link, mass 0.047177; collision cylinder length=0.06345282157546016 radius=0.02385968444719626; collision sphere radius=0.02385968444719626
- added link gripper_left_motor_double_link, mass 0.134356; collision cylinder length=0.044086614202536976 radius=0.056117638554986304; collision sphere radius=0.056117638554986304
- added link gripper_left_motor_single_dummy_mimic_link
- added link gripper_left_motor_single_link, mass 0.107923; collision cylinder length=0.018375470004515674 radius=0.06056680404353414; collision sphere radius=0.06056680404353414
- added link gripper_right_base_link, mass 0.637534; collision cylinder length=0.026984385527609595 radius=0.060646620008233225; collision sphere radius=0.060646620008233225
- added link gripper_right_inner_double_dummy_mimic_link
- added link gripper_right_inner_double_link, mass 0.087986; collision cylinder length=0.03702274994466908 radius=0.04877941290859063; collision sphere radius=0.04877941290859063
- added link gripper_right_inner_single_link, mass 0.047177; collision cylinder length=0.06345282157546016 radius=0.02385968444719626; collision sphere radius=0.02385968444719626
- added link gripper_right_link_dummy_mimic_link
- added link gripper_right_motor_double_link, mass 0.134356; collision cylinder length=0.044086614202536976 radius=0.056117638554986304; collision sphere radius=0.056117638554986304
- added link gripper_right_motor_single_dummy_mimic_link
- added link gripper_right_motor_single_link, mass 0.107923; collision cylinder length=0.018375470004515674 radius=0.06056680404353414; collision sphere radius=0.06056680404353414
- added link left_foot_lower_left
- added link left_foot_lower_right
- added link left_foot_upper_left
- added link left_foot_upper_right
- added link left_sole_link, mass 0.01
- added link leg_left_1_link, mass 2.235009; collision cylinder length=0.05831649869937837 radius=0.10038884516307987; collision sphere radius=0.10038884516307987
- added link leg_left_2_link, mass 1.490952; collision cylinder length=0.08642004451824492 radius=0.06522801409460995; collision sphere radius=0.06522801409460995
- added link leg_left_3_link, mass 6.239871; collision cylinder length=0.2927562662025252 radius=0.14557912147210253; collision sphere radius=0.14557912147210253
- added link leg_left_4_link, mass 3.759951; collision cylinder length=0.2946783341787494 radius=0.1184924950609377; collision sphere radius=0.1184924950609377
- added link leg_left_5_link, mass 1.29096; collision cylinder length=0.12378102303209611 radius=0.05628565171676146; collision sphere radius=0.05628565171676146
- added link leg_left_6_link, mass 1.597773; collision box size=0.21 0.13 0.02; visual mesh filename=v2/ankle_X_lo_res.stl scale=1 1 1
- added link leg_right_1_link, mass 2.235009; collision cylinder length=0.05831649869937837 radius=0.10038884516307987; collision sphere radius=0.10038884516307987
- added link leg_right_2_link, mass 1.490952; collision cylinder length=0.08642004451824492 radius=0.06522801409460995; collision sphere radius=0.06522801409460995
- added link leg_right_3_link, mass 6.239871; collision cylinder length=0.2927562662025252 radius=0.14557912147210253; collision sphere radius=0.14557912147210253
- added link leg_right_4_link, mass 3.759951; collision cylinder length=0.2946783341787494 radius=0.1184924950609377; collision sphere radius=0.1184924950609377
- added link leg_right_5_link, mass 1.29096; collision cylinder length=0.12378102303209611 radius=0.05628565171676146; collision sphere radius=0.05628565171676146
- added link leg_right_6_link, mass 1.597773; collision box size=0.21 0.13 0.02; visual mesh filename=v2/ankle_X_lo_res.stl scale=1 -1 1
- added link right_foot_lower_left
- added link right_foot_lower_right
- added link right_foot_upper_left
- added link right_foot_upper_right
- added link right_sole_link, mass 0.01
- added link wrist_left_ft_tool_link, mass 0.001; collision cylinder length=0.00975 radius=0.025; visual cylinder length=0.00975 radius=0.025
Joints:
- added joint gripper_left_base_link_joint: type fixed, parent wrist_left_ft_tool_link, child gripper_left_base_link, origin xyz=0.00000 0.00000 -0.02875 rpy=0.0 0.0 0.0, axis 0 0 0
- added joint gripper_left_fingertip_1_joint_mimic: type fixed, parent gripper_left_base_link, child gripper_left_fingertip_1_dummy_mimic_link
- added joint gripper_left_fingertip_2_joint_mimic: type fixed, parent gripper_left_base_link, child gripper_left_fingertip_2_dummy_mimic_link
- added joint gripper_left_fingertip_3_joint_mimic: type fixed, parent gripper_left_base_link, child gripper_left_fingertip_3_dummy_mimic_link
- added joint gripper_left_inner_double_joint: type revolute, parent gripper_left_base_link, child gripper_left_inner_double_link, origin xyz=0.00000 0.00525 -0.05598 rpy=0.0 0.0 0.0, axis 1 0 0, limit lower=-1.0471975511965976 upper=0.0 effort=100.0 velocity=1.0, mimic joint=gripper_left_joint multiplier=1.0 offset=0.0
- added joint gripper_left_inner_double_joint_mimic: type fixed, parent gripper_left_base_link, child gripper_left_inner_double_dummy_mimic_link
- added joint gripper_left_inner_single_joint: type revolute, parent gripper_left_base_link, child gripper_left_inner_single_link, origin xyz=0.00000 -0.00525 -0.05598 rpy=0.0 0.0 0.0, axis 1 0 0, limit lower=0.0 upper=1.0471975511965976 effort=100.0 velocity=1.0, mimic joint=gripper_left_joint multiplier=-1.0 offset=0.0
- added joint gripper_left_inner_single_joint_mimic: type fixed, parent gripper_left_base_link, child gripper_left_inner_single_dummy_mimic_link
- added joint gripper_left_joint: type revolute, parent gripper_left_base_link, child gripper_left_motor_double_link, origin xyz=0.0 0.02025 -0.03 rpy=0.0 0.0 0.0, axis 1 0 0, limit lower=-0.9599310885968813 upper=0.0 effort=1.0 velocity=1.0
- added joint gripper_left_motor_single_joint: type revolute, parent gripper_left_base_link, child gripper_left_motor_single_link, origin xyz=0.00000 -0.02025 -0.03000 rpy=0.0 0.0 0.0, axis 1 0 0, limit lower=0.0 upper=1.0471975511965976 effort=100.0 velocity=1.0, mimic joint=gripper_left_joint multiplier=-1.0 offset=0.0
- added joint gripper_left_motor_single_joint_mimic: type fixed, parent gripper_left_base_link, child gripper_left_motor_single_dummy_mimic_link
- added joint gripper_right_base_link_joint: type fixed, parent wrist_right_ft_tool_link, child gripper_right_base_link, origin xyz=0.00000 0.00000 -0.02875 rpy=0.0 0.0 0.0, axis 0 0 0
- added joint gripper_right_inner_double_joint: type revolute, parent gripper_right_base_link, child gripper_right_inner_double_link, origin xyz=0.00000 0.00525 -0.05598 rpy=0.0 0.0 0.0, axis 1 0 0, limit lower=-1.0471975511965976 upper=0.0 effort=100.0 velocity=1.0, mimic joint=gripper_right_joint multiplier=1.0 offset=0.0
- added joint gripper_right_inner_double_joint_mimic: type fixed, parent gripper_right_base_link, child gripper_right_inner_double_dummy_mimic_link
- added joint gripper_right_inner_single_joint: type revolute, parent gripper_right_base_link, child gripper_right_inner_single_link, origin xyz=0.00000 -0.00525 -0.05598 rpy=0.0 0.0 0.0, axis 1 0 0, limit lower=0.0 upper=1.0471975511965976 effort=100.0 velocity=1.0, mimic joint=gripper_right_joint multiplier=-1.0 offset=0.0
- added joint gripper_right_joint: type revolute, parent gripper_right_base_link, child gripper_right_motor_double_link, origin xyz=0.0 0.02025 -0.03 rpy=0.0 0.0 0.0, axis 1 0 0, limit lower=-0.9599310885968813 upper=0.0 effort=1.0 velocity=1.0
- added joint gripper_right_link_joint_mimic: type fixed, parent gripper_right_base_link, child gripper_right_link_dummy_mimic_link
- added joint gripper_right_motor_single_joint: type revolute, parent gripper_right_base_link, child gripper_right_motor_single_link, origin xyz=0.00000 -0.02025 -0.03000 rpy=0.0 0.0 0.0, axis 1 0 0, limit lower=0.0 upper=1.0471975511965976 effort=100.0 velocity=1.0, mimic joint=gripper_right_joint multiplier=-1.0 offset=0.0
- added joint gripper_right_motor_single_joint_mimic: type fixed, parent gripper_right_base_link, child gripper_right_motor_single_dummy_mimic_link
- added joint left_foot_lower_left_fix_joint: type fixed, parent left_sole_link, child left_foot_lower_left, origin xyz=-0.1 0.05 0.0 rpy=0 0 0
- added joint left_foot_lower_right_fix_joint: type fixed, parent left_sole_link, child left_foot_lower_right, origin xyz=-0.1 -0.05 0.0 rpy=0 0 0
- added joint left_foot_upper_left_fix_joint: type fixed, parent left_sole_link, child left_foot_upper_left, origin xyz=0.1 0.05 0.0 rpy=0 0 0
- added joint left_foot_upper_right_fix_joint: type fixed, parent left_sole_link, child left_foot_upper_right, origin xyz=0.1 -0.05 0.0 rpy=0 0 0
- added joint leg_left_1_joint: type revolute, parent base_link, child leg_left_1_link, origin xyz=-0.02 0.085 -0.27105 rpy=0.0 0.0 0.0, axis 0 0 1, limit lower=-0.3490658503988659 upper=1.5707963267948966 effort=100 velocity=3.87
- added joint leg_left_2_joint: type revolute, parent leg_left_1_link, child leg_left_2_link, origin xyz=0.0 0.0 0.0 rpy=0.0 0.0 0.0, axis 1 0 0, limit lower=-0.5236 upper=0.5236 effort=160 velocity=5.8
- added joint leg_left_3_joint: type revolute, parent leg_left_2_link, child leg_left_3_link, origin xyz=0.0 0.0 0.0 rpy=0.0 0.0 0.0, axis 0 1 0, limit lower=-2.095 upper=0.7 effort=160 velocity=5.8
- added joint leg_left_4_joint: type revolute, parent leg_left_3_link, child leg_left_4_link, origin xyz=0.0 0.0 -0.38 rpy=0.0 0.0 0.0, axis 0 1 0, limit lower=0 upper=2.618 effort=400 velocity=7
- added joint leg_left_5_joint: type revolute, parent leg_left_4_link, child leg_left_5_link, origin xyz=0.0 0.0 -0.325 rpy=0.0 0.0 0.0, axis 0 1 0, limit lower=-1.27 upper=0.68 effort=160 velocity=5.8
- added joint leg_left_6_joint: type revolute, parent leg_left_5_link, child leg_left_6_link, origin xyz=0.0 0.0 0.0 rpy=0.0 0.0 0.0, axis 1 0 0, limit lower=-0.5236 upper=0.5236 effort=100 velocity=4.8
- added joint leg_left_sole_fix_joint: type fixed, parent leg_left_6_link, child left_sole_link, origin xyz=0.00 0.00 -0.107 rpy=0 0 0, axis 1 0 0
- added joint leg_right_1_joint: type revolute, parent base_link, child leg_right_1_link, origin xyz=-0.02 -0.085 -0.27105 rpy=0.0 0.0 0.0, axis 0 0 1, limit lower=-1.5707963267948966 upper=0.3490658503988659 effort=100 velocity=3.87
- added joint leg_right_2_joint: type revolute, parent leg_right_1_link, child leg_right_2_link, origin xyz=0.0 0.0 0.0 rpy=0.0 0.0 0.0, axis 1 0 0, limit lower=-0.5236 upper=0.5236 effort=160 velocity=5.8
- added joint leg_right_3_joint: type revolute, parent leg_right_2_link, child leg_right_3_link, origin xyz=0.0 0.0 0.0 rpy=0.0 0.0 0.0, axis 0 1 0, limit lower=-2.095 upper=0.7 effort=160 velocity=5.8
- added joint leg_right_4_joint: type revolute, parent leg_right_3_link, child leg_right_4_link, origin xyz=0.0 0.0 -0.38 rpy=0.0 0.0 0.0, axis 0 1 0, limit lower=0 upper=2.618 effort=400 velocity=7
- added joint leg_right_5_joint: type revolute, parent leg_right_4_link, child leg_right_5_link, origin xyz=0.0 0.0 -0.325 rpy=0.0 0.0 0.0, axis 0 1 0, limit lower=-1.27 upper=0.68 effort=160 velocity=5.8
- added joint leg_right_6_joint: type revolute, parent leg_right_5_link, child leg_right_6_link, origin xyz=0.0 0.0 0.0 rpy=0.0 0.0 0.0, axis 1 0 0, limit lower=-0.5236 upper=0.5236 effort=100 velocity=4.8
- added joint leg_right_sole_fix_joint: type fixed, parent leg_right_6_link, child right_sole_link, origin xyz=0.00 0.00 -0.107 rpy=0 0 0, axis 1 0 0
- added joint right_foot_lower_left_fix_joint: type fixed, parent right_sole_link, child right_foot_lower_left, origin xyz=-0.1 0.05 0.0 rpy=0 0 0
- added joint right_foot_lower_right_fix_joint: type fixed, parent right_sole_link, child right_foot_lower_right, origin xyz=-0.1 -0.05 0.0 rpy=0 0 0
- added joint right_foot_upper_left_fix_joint: type fixed, parent right_sole_link, child right_foot_upper_left, origin xyz=0.1 0.05 0.0 rpy=0 0 0
- added joint right_foot_upper_right_fix_joint: type fixed, parent right_sole_link, child right_foot_upper_right, origin xyz=0.1 -0.05 0.0 rpy=0 0 0
- added joint wrist_left_tool_joint: type fixed, parent wrist_left_ft_link, child wrist_left_ft_tool_link, origin xyz=0 0 -0.012725 rpy=0 0 4.71238898038469
